File: RJ45_Connector_Port0.kicad_sch (KiCad schematic)
At the start: 13 parts, among them J1 0826-1X4T-43-F

Commit message: Adding page title, and confidential for now
Other:
- title: (none) -> RJ45 Connector Port 0 
Changed lines of the file:
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@@
 	(paper "A4")
 	(title_block
+		(title "RJ45 Connector Port 0 ")
 		(date "2025-12-21")
 		(rev "Rev. A")
 		(company "Kebag-Logic <contact@kebag-logic.com>")
+		(comment 1 "Confidential")
 	)
 	(junction

Commit message: fixes ERC errors in DC/DC converters
Parts:
- C24, C4, C5, C6: footprint Capacitor_SMD:C_0201_0603Metric -> KL_Footprints:C_0603; Dielectric X7R -> (none); Farnell 4539043 -> (none); Package_in_inch 0603 -> (none); Tolerance_in_pct 10 -> (none)
- C7: footprint Capacitor_SMD:C_0201_0603Metric -> KL_Footprints:C_0603
Changed lines of the file:
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@@
 		(fields_autoplaced yes)
 		(property "Reference" "C6"
-			(at 80.01 58.928 90)
+			(at 80.01 54.61 90)
 			(effects
 				(font
@@
 		)
 		(property "Value" "100n"
-			(at 80.01 65.532 90)
-			(effects
-				(font
-					(size 1.27 1.27)
-				)
-			)
-		)
-		(property "Footprint" "Capacitor_SMD:C_0201_0603Metric"
+			(at 80.01 57.15 90)
+			(effects
+				(font
+					(size 1.27 1.27)
+				)
+			)
+		)
+		(property "Footprint" "KL_Footprints:C_0603"
 			(at 76.2 63.1952 0)
 			(effects
@@
 		)
 		(property "LCSC" "C1591"
-			(at 80.01 62.23 0)
-			(effects
-				(font
-					(size 1.27 1.27)
-				)
-				(hide yes)
-			)
-		)
-		(property "Tolerance_in_pct" "10"
-			(at 80.01 62.23 0)
-			(effects
-				(font
-					(size 1.27 1.27)
-				)
-				(hide yes)
-			)
-		)
-		(property "Dielectric" "X7R"
-			(at 80.01 62.23 0)
-			(effects
-				(font
-					(size 1.27 1.27)
-				)
-				(hide yes)
-			)
-		)
-		(property "Package_in_inch" "0603"
-			(at 80.01 62.23 0)
-			(effects
-				(font
-					(size 1.27 1.27)
-				)
-				(hide yes)
-			)
-		)
-		(property "Farnell" "4539043"
 			(at 80.01 62.23 0)
 			(effects
@@
 		(fields_autoplaced yes)
 		(property "Reference" "C5"
-			(at 80.01 48.768 90)
+			(at 80.01 44.45 90)
 			(effects
 				(font
@@
 		)
 		(property "Value" "100n"
-			(at 80.01 55.626 90)
-			(effects
-				(font
-					(size 1.27 1.27)
-				)
-			)
-		)
-		(property "Footprint" "Capacitor_SMD:C_0201_0603Metric"
+			(at 80.01 46.99 90)
+			(effects
+				(font
+					(size 1.27 1.27)
+				)
+			)
+		)
+		(property "Footprint" "KL_Footprints:C_0603"
 			(at 83.82 51.1048 0)
 			(effects
@@
 		)
 		(property "LCSC" "C1591"
-			(at 80.01 52.07 0)
-			(effects
-				(font
-					(size 1.27 1.27)
-				)
-				(hide yes)
-			)
-		)
-		(property "Tolerance_in_pct" "10"
-			(at 80.01 52.07 0)
-			(effects
-				(font
-					(size 1.27 1.27)
-				)
-				(hide yes)
-			)
-		)
-		(property "Dielectric" "X7R"
-			(at 80.01 52.07 0)
-			(effects
-				(font
-					(size 1.27 1.27)
-				)
-				(hide yes)
-			)
-		)
-		(property "Package_in_inch" "0603"
-			(at 80.01 52.07 0)
-			(effects
-				(font
-					(size 1.27 1.27)
-				)
-				(hide yes)
-			)
-		)
-		(property "Farnell" "4539043"
 			(at 80.01 52.07 0)
 			(effects
@@
 			)
 		)
-		(property "Footprint" "Capacitor_SMD:C_0201_0603Metric"
+		(property "Footprint" "KL_Footprints:C_0603"
 			(at 110.1852 134.62 0)
 			(effects
@@
 		)
 		(property "LCSC" "C1591"
-			(at 109.22 130.81 0)
-			(effects
-				(font
-					(size 1.27 1.27)
-				)
-				(hide yes)
-			)
-		)
-		(property "Tolerance_in_pct" "10"
-			(at 109.22 130.81 0)
-			(effects
-				(font
-					(size 1.27 1.27)
-				)
-				(hide yes)
-			)
-		)
-		(property "Dielectric" "X7R"
-			(at 109.22 130.81 0)
-			(effects
-				(font
-					(size 1.27 1.27)
-				)
-				(hide yes)
-			)
-		)
-		(property "Package_in_inch" "0603"
-			(at 109.22 130.81 0)
-			(effects
-				(font
-					(size 1.27 1.27)
-				)
-				(hide yes)
-			)
-		)
-		(property "Farnell" "4539043"
 			(at 109.22 130.81 0)
 			(effects
@@
 		(fields_autoplaced yes)
 		(property "Reference" "C4"
-			(at 80.01 38.354 90)
+			(at 80.01 34.29 90)
 			(effects
 				(font
@@
 		)
 		(property "Value" "100n"
-			(at 80.01 45.212 90)
-			(effects
-				(font
-					(size 1.27 1.27)
-				)
-			)
-		)
-		(property "Footprint" "Capacitor_SMD:C_0201_0603Metric"
+			(at 80.01 36.83 90)
+			(effects
+				(font
+					(size 1.27 1.27)
+				)
+			)
+		)
+		(property "Footprint" "KL_Footprints:C_0603"
 			(at 83.82 40.9448 0)
 			(effects
@@
 		)
 		(property "LCSC" "C1591"
-			(at 80.01 41.91 0)
-			(effects
-				(font
-					(size 1.27 1.27)
-				)
-				(hide yes)
-			)
-		)
-		(property "Tolerance_in_pct" "10"
-			(at 80.01 41.91 0)
-			(effects
-				(font
-					(size 1.27 1.27)
-				)
-				(hide yes)
-			)
-		)
-		(property "Dielectric" "X7R"
-			(at 80.01 41.91 0)
-			(effects
-				(font
-					(size 1.27 1.27)
-				)
-				(hide yes)
-			)
-		)
-		(property "Package_in_inch" "0603"
-			(at 80.01 41.91 0)
-			(effects
-				(font
-					(size 1.27 1.27)
-				)
-				(hide yes)
-			)
-		)
-		(property "Farnell" "4539043"
 			(at 80.01 41.91 0)
 			(effects
@@
 		(fields_autoplaced yes)
 		(property "Reference" "C7"
-			(at 80.01 69.088 90)
+			(at 80.01 64.77 90)
 			(effects
 				(font
@@
 		)
 		(property "Value" "100n"
-			(at 80.01 75.692 90)
-			(effects
-				(font
-					(size 1.27 1.27)
-				)
-			)
-		)
-		(property "Footprint" "Capacitor_SMD:C_0201_0603Metric"
+			(at 80.01 67.31 90)
+			(effects
+				(font
+					(size 1.27 1.27)
+				)
+			)
+		)
+		(property "Footprint" "KL_Footprints:C_0603"
 			(at 83.82 73.3552 0)
 			(effects

Commit message: updates components from my library misconfiguration. Refs: #1
Parts:
- J1: footprint 0826-1X4T-43-F:BEL_0826-1X4T-43-F -> KL_Footprints:BEL_0826-1X4T-43-F
- R5, R6, R7, R75, R76, R77, R78: footprint KL_Footprints:C_0603 -> KL_Footprints:R_0603
Changed lines of the file:
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@@
 		(fields_autoplaced yes)
 		(property "Reference" "R6"
-			(at 119.38 77.724 90)
+			(at 119.38 73.66 90)
 			(effects
 				(font
@@
 		)
 		(property "Value" "1K"
-			(at 119.38 82.55 90)
-			(effects
-				(font
-					(size 1.27 1.27)
-				)
-			)
-		)
-		(property "Footprint" "KL_Footprints:C_0603"
+			(at 119.38 76.2 90)
+			(effects
+				(font
+					(size 1.27 1.27)
+				)
+			)
+		)
+		(property "Footprint" "KL_Footprints:R_0603"
 			(at 119.38 81.788 90)
 			(effects
@@
 			)
 		)
-		(property "Footprint" "KL_Footprints:C_0603"
+		(property "Footprint" "KL_Footprints:R_0603"
 			(at 114.808 114.3 90)
 			(effects
@@
 			)
 		)
-		(property "Footprint" "KL_Footprints:C_0603"
+		(property "Footprint" "KL_Footprints:R_0603"
 			(at 97.028 114.3 90)
 			(effects
@@
 			)
 		)
-		(property "Footprint" "KL_Footprints:C_0603"
+		(property "Footprint" "KL_Footprints:R_0603"
 			(at 79.502 114.3 90)
 			(effects
@@
 			)
 		)
-		(property "Footprint" "KL_Footprints:C_0603"
+		(property "Footprint" "KL_Footprints:R_0603"
 			(at 123.698 114.3 90)
 			(effects
@@
 			)
 		)
-		(property "Footprint" "KL_Footprints:C_0603"
+		(property "Footprint" "KL_Footprints:R_0603"
 			(at 105.918 114.3 90)
 			(effects
@@
 			)
 		)
-		(property "Footprint" "0826-1X4T-43-F:BEL_0826-1X4T-43-F"
+		(property "Footprint" "KL_Footprints:BEL_0826-1X4T-43-F"
 			(at 139.7 69.85 0)
 			(effects
@@
 			)
 		)
-		(property "Footprint" "KL_Footprints:C_0603"
+		(property "Footprint" "KL_Footprints:R_0603"
 			(at 79.502 100.33 90)
 			(effects

Commit message: removes unused busses, adds cheaper 0R resistor, clean up to fix ERC errors. Refs: #1
Changed lines of the file:
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@@
 		(on_board yes)
 		(dnp no)
-		(fields_autoplaced yes)
 		(property "Reference" "R6"
-			(at 119.38 73.66 90)
+			(at 119.38 77.978 90)
 			(effects
 				(font
@@
 		)
 		(property "Value" "1K"
-			(at 119.38 76.2 90)
+			(at 119.38 82.55 90)
 			(effects
 				(font
