File: RJ45_Connector_Port0.kicad_sch (KiCad schematic)
At the start: 13 parts, among them J1 RJ45_0826-1X4T-43-F

Commit message: connects the shield pins to GND. Refs: #50
Parts:
- removed C24: 100n, KL_Footprints:C_0603, symbol KL_C:C_100n_50V_10pct_X7R_0603
- removed R75, R76, R77, R78: 330R, KL_Footprints:R_0603, symbol KL_R:R_330R_0.1W_1pct_0603
Connections:
- net GND: now also J1.S1 (SHIELD), J1.S2 (SHIELD__1), J1.S3 (SHIELD__2), J1.S4 (SHIELD__3)
