File: switch_phys.kicad_sch (KiCad schematic)
At the start: 2 parts

Commit message: updates components from my library misconfiguration. Refs: #1
Parts:
- R70: footprint KL_Footprints:C_0603 -> KL_Footprints:R_0603
- U1: footprint Package_QFP:TQFP-128_14x14mm_P0.4mm -> KL_Footprints:TQFP-128_14x14mm_P0.4mm
Changed lines of the file:
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@@
 			)
 		)
-		(property "Footprint" "KL_Footprints:C_0603"
+		(property "Footprint" "KL_Footprints:R_0603"
 			(at 16.002 67.31 90)
 			(effects
@@
 		(fields_autoplaced yes)
 		(property "Reference" "U1"
-			(at 43.18 162.56 0)
+			(at 43.18 54.61 0)
 			(effects
 				(font
@@
 			)
 		)
-		(property "Footprint" "Package_QFP:TQFP-128_14x14mm_P0.4mm"
+		(property "Footprint" "KL_Footprints:TQFP-128_14x14mm_P0.4mm"
 			(at 39.878 183.642 0)
 			(effects

Commit message: consistent naming for hierarchical pin and attached net. Refs: #1
Changed lines of the file:
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@@
 	(wire
 		(pts
-			(xy 19.05 16.51) (xy 29.21 16.51)
+			(xy 22.86 16.51) (xy 33.02 16.51)
 		)
 		(stroke
@@
 	)
 	(label "3V3_PHY"
-		(at 29.21 16.51 180)
+		(at 33.02 16.51 180)
 		(effects
 			(font
@@
 		)
 	)
-	(hierarchical_label "3V3"
+	(hierarchical_label "3V3_PHY"
 		(shape input)
-		(at 19.05 16.51 180)
-		(effects
-			(font
+		(at 22.86 16.51 180)
+		(effects
+			(font
