File: switch_phys.kicad_sch (KiCad schematic)
At the start: 2 parts

Commit message: updates component details for ordering. Refs: #1
Parts:
- U1: value ~ -> LAN96455F-I/8MW; Digikey (none) -> 150-LAN96455F-I/8MW-ND; Mouser (none) -> 579-LAN96455FI8MW; manf# LAN96455F-I/8MW -> (none)
Changed lines of the file:
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@@
+			)
+		)
+		(property "Dielectric" ""
+			(at 17.78 67.31 0)
+			(effects
+				(font
+					(size 1.27 1.27)
+				)
+				(hide yes)
+			)
+		)
+		(property "Dielectric_type" ""
+			(at 17.78 67.31 0)
+			(effects
+				(font
+					(size 1.27 1.27)
+				)
+				(hide yes)
+			)
+		)
+		(property "LSCS" ""
+			(at 17.78 67.31 0)
+			(effects
+				(font
+					(size 1.27 1.27)
+				)
+				(hide yes)
+			)
+		)
+		(property "Max Current" ""
+			(at 17.78 67.31 0)
+			(effects
+				(font
+					(size 1.27 1.27)
+				)
+				(hide yes)
 			)
 		)
@@
 			)
 		)
-		(property "Value" "~"
+		(property "Value" "LAN96455F-I/8MW"
 			(at 55.88 143.51 0)
 			(effects
@@
 			)
 		)
-		(property "manf#" "LAN96455F-I/8MW"
-			(at 40.64 169.418 0)
+		(property "Mouser" "579-LAN96455FI8MW"
+			(at 55.88 160.02 0)
 			(effects
 				(font
+					(size 1.27 1.27)
+				)
+				(hide yes)
+			)
+		)
+		(property "Digikey" "150-LAN96455F-I/8MW-ND"
+			(at 55.88 160.02 0)
+			(effects
+				(font
+					(size 1.27 1.27)
+				)
+				(hide yes)
+			)
+		)
+		(property "LCSC" ""
+			(at 55.88 160.02 0)
+			(effects
+				(font

Commit message: initial commit for automatic current consumption calculation. Refs: #9
Parts:
- U1: I_DD_1V15_max_A (none) -> 0.935; I_DD_AH25_2V5_max_A (none) -> 0.475; I_DD_AH33_3V3_max_A (none) -> 0.505; I_DD_ALSx_1V15_max_A (none) -> 0.025; I_DD_AL_1V15_max_A (none) -> 0.400; I_DD_IO25_2V5_max_A (none) -> 0.045; I_DD_IO33_3V3_max_A (none) -> 0.075; I_DD_IOD (none) -> 0.005
Changed lines of the file:
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@@
+			)
+		)
+		(property "I_DD_1V15_max_A" "0.935"
+			(at 55.88 160.02 0)
+			(effects
+				(font
+					(size 1.27 1.27)
+				)
+				(hide yes)
+			)
+		)
+		(property "I_DD_AL_1V15_max_A" "0.400"
+			(at 55.88 160.02 0)
+			(effects
+				(font
+					(size 1.27 1.27)
+				)
+				(hide yes)
+			)
+		)
+		(property "I_DD_ALSx_1V15_max_A" "0.025"
+			(at 55.88 160.02 0)
+			(effects
+				(font
+					(size 1.27 1.27)
+				)
+				(hide yes)
+			)
+		)
+		(property "I_DD_AH25_2V5_max_A" "0.475"
+			(at 55.88 160.02 0)
+			(effects
+				(font
+					(size 1.27 1.27)
+				)
+				(hide yes)
+			)
+		)
+		(property "I_DD_AH33_3V3_max_A" "0.505"
+			(at 55.88 160.02 0)
+			(effects
+				(font
+					(size 1.27 1.27)
+				)
+				(hide yes)
+			)
+		)
+		(property "I_DD_IO25_2V5_max_A" "0.045"
+			(at 55.88 160.02 0)
+			(effects
+				(font
+					(size 1.27 1.27)
+				)
+				(hide yes)
+			)
+		)
+		(property "I_DD_IO33_3V3_max_A" "0.075"
+			(at 55.88 160.02 0)
+			(effects
+				(font
+					(size 1.27 1.27)
+				)
+				(hide yes)
+			)
+		)
+		(property "I_DD_IOD" "0.005"
+			(at 55.88 160.02 0)
+			(effects
+				(font
+					(size 1.27 1.27)
+				)
+				(hide yes)
 			)
 		)

Commit message: updates switch_phys. Refs: #41
Parts:
- R70: symbol KL_R:R_6K04_100mw_001_0603 -> KL_R:R_6K04_0.1W_1pct_0603; MPN (none) -> RMCF0603FT6K04; Package (in) 0603 -> (none); Package_in_inch (none) -> 0603; Power 100mW -> (none); Power_in_W (none) -> 0.1; Tolerance 1% -> (none); Tolerance_in_pct (none) -> 1
- U1: symbol KL_IC_LAN9645xF:lan9645xF_128_TQFP -> KL_Network_Switch:LAN96455F_TQFP-128; LCSC (none) -> NA; MPN (none) -> LAN96455F-I/8MW
Changed lines of the file:
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@@
 	)
 	(symbol
-		(lib_id "KL_R:R_6K04_100mw_001_0603")
+		(lib_id "KL_R:R_6K04_0.1W_1pct_0603")
 		(at 17.78 67.31 0)
 		(unit 1)
@@
 			)
 		)
-		(property "Datasheet" ""
+		(property "Datasheet" "https://www.seielect.com/catalog/sei-rmcf_rmcp.pdf"
 			(at 17.78 67.31 0)
 			(hide yes)
@@
 			)
 		)
-		(property "Power" "100mW"
-			(at 17.78 67.31 0)
-			(hide yes)
-			(show_name no)
-			(do_not_autoplace no)
-			(effects
-				(font
-					(size 1.27 1.27)
-				)
-			)
-		)
-		(property "Tolerance" "1%"
-			(at 17.78 67.31 0)
-			(hide yes)
-			(show_name no)
-			(do_not_autoplace no)
-			(effects
-				(font
-					(size 1.27 1.27)
-				)
-			)
-		)
 		(property "Mouser" "708-RMCF0603FT6K04"
 			(at 17.78 67.31 0)
@@
 			)
 		)
-		(property "Farnell" ""
-			(at 17.78 67.31 0)
-			(hide yes)
-			(show_name no)
-			(do_not_autoplace no)
-			(effects
-				(font
-					(size 1.27 1.27)
-				)
-			)
-		)
-		(property "Package (in)" "0603"
+		(property "Power_in_W" "0.1"
+			(at 17.78 67.31 0)
+			(hide yes)
+			(show_name no)
+			(do_not_autoplace no)
+			(effects
+				(font
+					(size 1.27 1.27)
+				)
+			)
+		)
+		(property "Tolerance_in_pct" "1"
+			(at 17.78 67.31 0)
+			(hide yes)
+			(show_name no)
+			(do_not_autoplace no)
+			(effects
+				(font
+					(size 1.27 1.27)
+				)
+			)
+		)
+		(property "MPN" "RMCF0603FT6K04"
+			(at 17.78 67.31 0)
+			(hide yes)
+			(show_name no)
+			(do_not_autoplace no)
+			(effects
+				(font
+					(size 1.27 1.27)
+				)
+			)
+		)
+		(property "Package_in_inch" "0603"
 			(at 17.78 67.31 0)
 			(hide yes)
@@
 	)
 	(symbol
-		(lib_id "KL_IC_LAN9645xF:lan9645xF_128_TQFP")
+		(lib_id "KL_Network_Switch:LAN96455F_TQFP-128")
 		(at 55.88 160.02 180)
 		(unit 3)
@@
 			)
 		)
-		(property "Datasheet" ""
+		(property "Datasheet" "https://ww1.microchip.com/downloads/aemDocuments/documents/NCS/ProductDocuments/DataSheets/LAN9645xF_Data_Sheet_DS00006065.pdf"
 			(at 55.88 143.51 0)
 			(hide yes)
@@
 			)
 		)
-		(property "Description" ""
+		(property "Description" "Network Switch"
 			(at 55.88 143.51 0)
 			(hide yes)
@@
 			)
 		)
-		(property "LCSC" ""
+		(property "LCSC" "NA"
 			(at 55.88 160.02 0)
 			(hide yes)
@@
 		)
 		(property "I_DD_IOD" "0.005"
+			(at 55.88 160.02 0)
+			(hide yes)
+			(show_name no)
+			(do_not_autoplace no)
+			(effects
+				(font
+					(size 1.27 1.27)
+				)
+			)
+		)
+		(property "MPN" "LAN96455F-I/8MW "
 			(at 55.88 160.02 0)
 			(hide yes)
@@
 			)
 			(project "shish-lan"
-				(path "/d4536448-b109-4159-96e2-3dc21baf2d6e/0b7d9af9-83c1-43fa-a7a0-a33d0a00ea9c/7f5fd65f-f670-4db7-8f09-63d4fb2faa09"
-					(reference "U1")
-					(unit 3)
-				)
 				(path "/d4536448-b109-4159-96e2-3dc21baf2d6e/0b7d9af9-83c1-43fa-a7a0-a33d0a00ea9c/cbb6064c-9387-4840-bb4d-7326af14ff9d"
 					(reference "U1")
 					(unit 3)
 				)
-				(path "/d4536448-b109-4159-96e2-3dc21baf2d6e/0b7d9af9-83c1-43fa-a7a0-a33d0a00ea9c/d7edf10b-e7e7-437a-ab6c-966f29ad8f7f"
-					(reference "U1")
-					(unit 3)
-				)
 			)
 		)
 	)
 	(symbol
-		(lib_id "KL_SYM_LOCAL:GND")
+		(lib_id "power:GND")
 		(at 17.78 73.66 0)
 		(unit 1)
