File: switch_gpio_config.kicad_sch (KiCad schematic)
At the start: 44 parts

Commit message: updates switch_gpio_config. Refs: #41
Parts:
- R14, R26, R27, R28, R29, R30, R31, R32, R33, R34, R35, R36, R37, R38, R39, R40, R41, R42, R43, R44, R45, R46, R47, R48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: symbol KL_R:R_10K_100mW_5_0603 -> KL_R:R_10K_0.1W_5pct_0603; MPN (none) -> CRCW060310K0JNEC; Package (in) 0603 -> (none); Package_in_inch (none) -> 0603; Power 100mW -> (none); Power_in_W (none) -> 0.1; Tolerance 5% -> (none); Tolerance_in_pct (none) -> 5
