File: switch_gpio_config.kicad_sch (KiCad schematic)
At the start: 44 parts

Commit message: Pull JTAG_ENB high: fit R41, DNP R53
Refs #79
Parts:
- R41: now fitted
- R53: now not fitted
Connections:
- net JTAG_EN renamed JTAG_ENB

Commit message: Udpate text to not confuse people Refs: #79
Other:
- note added: "Note: If JTAG is enabled, configuration strap BOOT_MODE0 selects: 0: DFT TAP controller 1: SerDes TAP controller 0: Enable JTAG *1: Disable JTAG"
- note removed: "Note: If JTAG is enabled, configuration strap BOOT_MODE0 selects: 0: DFT TAP controller 1: SerDes TAP controller *0: Disable JTAG 1: Enable JTAG"

Commit message: Managed mode: boot 000, DNP unmanaged straps
Refs #62
Parts:
- R26, R28, R30, R31, R33, R34, R42, R46, R48, R49, R51, R57, R59, R60, R64: now not fitted
- R52, R68: now fitted
Changed lines of the file:
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@@
 		(on_board yes)
 		(in_pos_files yes)
-		(dnp no)
+		(dnp yes)
 		(fields_autoplaced yes)
 		(property "Reference" "R42"
@@
 		(on_board yes)
 		(in_pos_files yes)
-		(dnp no)
+		(dnp yes)
 		(fields_autoplaced yes)
 		(property "Reference" "R26"
@@
 		(on_board yes)
 		(in_pos_files yes)
-		(dnp yes)
+		(dnp no)
 		(fields_autoplaced yes)
 		(property "Reference" "R52"
@@
 		(on_board yes)
 		(in_pos_files yes)
-		(dnp no)
+		(dnp yes)
 		(fields_autoplaced yes)
 		(property "Reference" "R59"
@@
 		(on_board yes)
 		(in_pos_files yes)
-		(dnp no)
+		(dnp yes)
 		(fields_autoplaced yes)
 		(property "Reference" "R49"
@@
 		(on_board yes)
 		(in_pos_files yes)
-		(dnp no)
+		(dnp yes)
 		(fields_autoplaced yes)
 		(property "Reference" "R34"
@@
 		(on_board yes)
 		(in_pos_files yes)
-		(dnp no)
+		(dnp yes)
 		(fields_autoplaced yes)
 		(property "Reference" "R48"
@@
 		(on_board yes)
 		(in_pos_files yes)
-		(dnp yes)
+		(dnp no)
 		(fields_autoplaced yes)
 		(property "Reference" "R68"
@@
 		(on_board yes)
 		(in_pos_files yes)
-		(dnp no)
+		(dnp yes)
 		(fields_autoplaced yes)
 		(property "Reference" "R30"
@@
 		(on_board yes)
 		(in_pos_files yes)
-		(dnp no)
+		(dnp yes)
 		(fields_autoplaced yes)
 		(property "Reference" "R64"
@@
 		(on_board yes)
 		(in_pos_files yes)
-		(dnp no)
+		(dnp yes)
 		(fields_autoplaced yes)
 		(property "Reference" "R57"
@@
 		(on_board yes)
 		(in_pos_files yes)
-		(dnp no)
+		(dnp yes)
 		(fields_autoplaced yes)
 		(property "Reference" "R60"
@@
 		(on_board yes)
 		(in_pos_files yes)
-		(dnp no)
+		(dnp yes)
 		(fields_autoplaced yes)
 		(property "Reference" "R51"
@@
 		(on_board yes)
 		(in_pos_files yes)
-		(dnp no)
+		(dnp yes)
 		(fields_autoplaced yes)
 		(property "Reference" "R31"
@@
 		(on_board yes)
 		(in_pos_files yes)
-		(dnp no)
+		(dnp yes)
 		(fields_autoplaced yes)
 		(property "Reference" "R28"
@@
 		(on_board yes)
 		(in_pos_files yes)
-		(dnp no)
+		(dnp yes)
 		(fields_autoplaced yes)
 		(property "Reference" "R46"
@@
 		(on_board yes)
 		(in_pos_files yes)
-		(dnp no)
+		(dnp yes)
 		(fields_autoplaced yes)
 		(property "Reference" "R33"

Commit message: Boot mode note: mark managed (0) as default
Refs #62
Other:
- note added: "Boot Mode Selector Note: Unmanaged modes are selected using options 3, 4, 5, 6, or 7. *0: [Managed] No boot --> Need management interface to work 1: RESERVED 2: RESERVED 3: [Unmanaged] ROM boot. 4: [Unmanaged] ROM + I2C table boot. 5: [Unmanaged] ROM + SPI table boot. 6: [Unmanaged] ROM + VRAP port 5 boot. 7: [Unmanaged] ROM + VRAP port 7 boot."
- note removed: "Boot Mode Selector Note: Unmanaged modes are selected using options 3, 4, 5, 6, or 7. 0: [Managed] No boot --> Need management interface to work 1: RESERVED 2: RESERVED *3: [Unmanaged] ROM boot. 4: [Unmanaged] ROM + I2C table boot. 5: [Unmanaged] ROM + SPI table boot. 6: [Unmanaged] ROM + VRAP port 5 boot. 7: [Unmanaged] ROM + VRAP port 7 boot."
Changed lines of the file:
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@@
 		)
 	)
-	(text "Boot Mode Selector\nNote: Unmanaged modes are  selected using\noptions 3, 4,  5, 6, or 7.\n0: [Managed] No boot --> Need management interface to work\n1: RESERVED\n2: RESERVED\n*3: [Unmanaged] ROM boot.\n4:  [Unmanaged] ROM + I2C table boot.\n5:  [Unmanaged] ROM + SPI table boot.\n6:  [Unmanaged] ROM + VRAP port 5 boot. \n7:  [Unmanaged] ROM + VRAP port 7 boot. "
+	(text "Boot Mode Selector\nNote: Unmanaged modes are  selected using\noptions 3, 4,  5, 6, or 7.\n*0: [Managed] No boot --> Need management interface to work\n1: RESERVED\n2: RESERVED\n3: [Unmanaged] ROM boot.\n4:  [Unmanaged] ROM + I2C table boot.\n5:  [Unmanaged] ROM + SPI table boot.\n6:  [Unmanaged] ROM + VRAP port 5 boot. \n7:  [Unmanaged] ROM + VRAP port 7 boot. "
 		(exclude_from_sim no)
 		(at 15.494 33.782 0)
