File: stm_dbg_header.kicad_sch (KiCad schematic)
At the start: 1 part, among them J11 02x10_2.54mm_Header_Odd_Even

Commit message: updates component details for ordering. Refs: #1
Parts:
- J11: Digikey (none) -> 2057-BHR-20-VUA-ND; LCSC (none) -> C598987; Mouser (none) -> 737-BHR-20-VUA
Changed lines of the file:
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@@
+			)
+		)
+		(property "Manufacturer_No" ""
+			(at 123.19 85.09 0)
+			(effects
+				(font
+					(size 1.27 1.27)
+				)
+				(hide yes)
+			)
+		)
+		(property "Mouser" "737-BHR-20-VUA"
+			(at 123.19 85.09 0)
+			(effects
+				(font
+					(size 1.27 1.27)
+				)
+				(hide yes)
+			)
+		)
+		(property "Digikey" "2057-BHR-20-VUA-ND"
+			(at 123.19 85.09 0)
+			(effects
+				(font
+					(size 1.27 1.27)
+				)
+				(hide yes)
+			)
+		)
+		(property "LCSC" "C598987"
+			(at 123.19 85.09 0)
+			(effects
+				(font
+					(size 1.27 1.27)
+				)
+				(hide yes)
 			)
 		)

Commit message: updates stm_dbg_header. Refs: #41
Parts:
- J11: value 02x10_2.54mm_Header_Odd_Even -> Header_10x02_2.54mm_2.54mm_Straight; symbol KL_Headers:02x10_2.54mm_Header_Odd_Even -> KL_Header:Header_10x02_2.54mm_2.54mm_Straight; MPN (none) -> BHR-20-VUA; No_of_pins (none) -> 10; No_of_rows (none) -> 2; Orientation (none) -> Straight; Pitch_pin_in_mm (none) -> 2.54; Pitch_row_in_mm (none) -> 2.54
Changed lines of the file:
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@@
 	)
 	(symbol
-		(lib_id "KL_Headers:02x10_2.54mm_Header_Odd_Even")
+		(lib_id "KL_Header:Header_10x02_2.54mm_2.54mm_Straight")
 		(at 123.19 85.09 0)
 		(unit 1)
@@
 			)
 		)
-		(property "Value" "02x10_2.54mm_Header_Odd_Even"
+		(property "Value" "Header_10x02_2.54mm_2.54mm_Straight"
 			(at 124.46 100.33 0)
 			(hide yes)
@@
 			)
 		)
-		(property "Datasheet" ""
+		(property "Datasheet" "https://app.adam-tech.com/products/download/data_sheet/203218/bhr-xx-vua-data-sheet.pdf"
 			(at 123.19 85.09 0)
 			(hide yes)
@@
 			)
 		)
-		(property "Description" "Generic connector, double row, 02x10, odd/even pin numbering scheme (row 1 odd numbers, row 2 even numbers), script generated (kicad-library-utils/schlib/autogen/connector/)"
-			(at 123.19 85.09 0)
-			(hide yes)
-			(show_name no)
-			(do_not_autoplace no)
-			(effects
-				(font
-					(size 1.27 1.27)
-				)
-			)
-		)
-		(property "Manufacturer_No" ""
+		(property "Description" "Pin header"
 			(at 123.19 85.09 0)
 			(hide yes)
@@
 			(at 123.19 85.09 0)
 			(hide yes)
+			(show_name no)
+			(do_not_autoplace no)
+			(effects
+				(font
+					(size 1.27 1.27)
+				)
+			)
+		)
+		(property "No_of_pins" "10"
+			(at 123.19 85.09 0)
+			(hide yes)
+			(show_name no)
+			(do_not_autoplace no)
+			(effects
+				(font
+					(size 1.27 1.27)
+				)
+			)
+		)
+		(property "No_of_rows" "2"
+			(at 123.19 85.09 0)
+			(hide yes)
+			(show_name no)
+			(do_not_autoplace no)
+			(effects
+				(font
+					(size 1.27 1.27)
+				)
+			)
+		)
+		(property "Pitch_pin_in_mm" "2.54"
+			(at 123.19 85.09 0)
+			(hide yes)
+			(show_name no)
+			(do_not_autoplace no)
+			(effects
+				(font
+					(size 1.27 1.27)
+				)
+			)
+		)
+		(property "Pitch_row_in_mm" "2.54"
+			(at 123.19 85.09 0)
+			(hide yes)
+			(show_name no)
+			(do_not_autoplace no)
+			(effects
+				(font
+					(size 1.27 1.27)
+				)
+			)
+		)
+		(property "Orientation" "Straight"
+			(at 123.19 85.09 0)
+			(hide yes)
+			(show_name no)
+			(do_not_autoplace no)
+			(effects
+				(font
+					(size 1.27 1.27)
+				)
+			)
+		)
+		(property "MPN" "BHR-20-VUA"
+			(at 123.19 85.09 0)
+			(hide yes)
