File: crystal.kicad_sch (KiCad schematic)
At the start: 3 parts, among them X2 25000000

Commit message: adds footprint for VXM7. Refs: #1
Parts:
- X2: footprint (none) -> KL_Footprints:VXM7
Changed lines of the file:
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@@
 			)
 		)
-		(property "Footprint" ""
+		(property "Footprint" "KL_Footprints:VXM7"
 			(at 142.24 95.25 0)
 			(effects

Commit message: 1: adding crystal sheet name
Other:
- title: (none) -> Oscillator 25MHz
Changed lines of the file:
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@@
 	(paper "A4")
 	(title_block
+		(title "Oscillator 25MHz")
 		(date "2025-12-14")
 		(rev "rev A")
 		(company "Kebag-logic <contact@kebag-logic.com>")
+		(comment 1 "Confidential")
 	)
 	(junction

Commit message: updates symbols and fixes ERC errors. Refs: #9
Changed lines of the file:
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@@
 		(fields_autoplaced yes)
 		(property "Reference" "C92"
-			(at 138.43 107.95 90)
+			(at 138.43 95.25 90)
 			(effects
 				(font
@@
 		)
 		(property "Value" "10p"
-			(at 138.43 110.49 90)
+			(at 138.43 97.79 90)
 			(effects
 				(font
@@
 		(property "LCSC" "C2229848"
 			(at 138.43 102.87 0)
-			(effects
-				(font
-					(size 1.27 1.27)
-				)
-				(hide yes)
-			)
-		)
-		(property "Dielectric" ""
-			(at 138.43 102.87 90)
-			(effects
-				(font
-					(size 1.27 1.27)
-				)
-				(hide yes)
-			)
-		)
-		(property "Dielectric_type" ""
-			(at 138.43 102.87 90)
-			(effects
-				(font
-					(size 1.27 1.27)
-				)
-				(hide yes)
-			)
-		)
-		(property "LSCS" ""
-			(at 138.43 102.87 90)
-			(effects
-				(font
-					(size 1.27 1.27)
-				)
-				(hide yes)
-			)
-		)
-		(property "Max Current" ""
-			(at 138.43 102.87 90)
 			(effects
 				(font
@@
 			)
 		)
-		(property "Dielectric" ""
-			(at 138.43 88.9 90)
-			(effects
-				(font
-					(size 1.27 1.27)
-				)
-				(hide yes)
-			)
-		)
-		(property "Dielectric_type" ""
-			(at 138.43 88.9 90)
-			(effects
-				(font
-					(size 1.27 1.27)
-				)
-				(hide yes)
-			)
-		)
-		(property "LSCS" ""
-			(at 138.43 88.9 90)
-			(effects
-				(font
-					(size 1.27 1.27)
-				)
-				(hide yes)
-			)
-		)
-		(property "Max Current" ""
-			(at 138.43 88.9 90)
-			(effects
-				(font
-					(size 1.27 1.27)
-				)
-				(hide yes)
-			)
-		)
 		(pin "2"
 		)
@@
 				(hide yes)
 			)
-		)
-		(property "Dielectric" ""
-			(at 142.24 95.25 90)
-			(effects
-				(font
-					(size 1.27 1.27)
-				)
-				(hide yes)
-			)
-		)
-		(property "Dielectric_type" ""
-			(at 142.24 95.25 90)
-			(effects
-				(font
-					(size 1.27 1.27)
-				)
-				(hide yes)
-			)
-		)
-		(property "LSCS" ""
-			(at 142.24 95.25 90)
-			(effects
-				(font
-					(size 1.27 1.27)
-				)
-				(hide yes)
-			)
-		)
-		(property "Max Current" ""
-			(at 142.24 95.25 90)
-			(effects
-				(font
-					(size 1.27 1.27)
-				)
-				(hide yes)
-			)

Commit message: updates components to latest library. Refs: #30
Changed lines of the file:
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@@
 		(fields_autoplaced yes)
 		(property "Reference" "C92"
-			(at 138.43 95.25 90)
+			(at 138.43 107.95 90)
 			(effects
 				(font
@@
 		)
 		(property "Value" "10p"
-			(at 138.43 97.79 90)
+			(at 138.43 110.49 90)
 			(effects
 				(font

Commit message: updates crystal. Refs: #41
Parts:
- C86, C92: symbol KL_C:C_10p_25V_C0G_0603_5 -> KL_C:C_10p_25V_5pct_C0G_0603; Dielectric (none) -> C0G; MPN (none) -> 06033U100JAT2A; Package_in_inch (none) -> 0603; Tolerance 5 -> (none); Tolerance_in_pct (none) -> 5; Voltage 25V -> (none); Voltage_in_V (none) -> 25
- X2: value 25000000 -> 25M; symbol KL_Passive_ICs:Crystal_25MHz_32p -> KL_Crystal:Crystal_25M_10ppm_32pF_3.2x2.5; Frequency_Tolerance_in_ppm (none) -> 10; Load_Capacitance_in_pF (none) -> 32; MPN (none) -> VXM7-9032-25M0000000; Package_LxW_in_mm (none) -> 3.2x2.5
Changed lines of the file:
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@@
 	)
 	(symbol
-		(lib_id "KL_SYM_LOCAL:GND")
+		(lib_id "power:GND")
 		(at 132.08 95.25 0)
 		(unit 1)
@@
 	)
 	(symbol
-		(lib_id "KL_C:C_10p_25V_C0G_0603_5")
+		(lib_id "KL_C:C_10p_25V_5pct_C0G_0603")
 		(at 138.43 102.87 270)
 		(unit 1)
@@
 			)
 		)
-		(property "Datasheet" ""
+		(property "Datasheet" "https://datasheets.kyocera-avx.com/U-Series.pdf"
 			(at 138.43 102.87 0)
 			(hide yes)
@@
 			)
 		)
-		(property "Tolerance" "5"
-			(at 138.43 102.87 0)
-			(hide yes)
-			(show_name no)
-			(do_not_autoplace no)
-			(effects
-				(font
-					(size 1.27 1.27)
-				)
-			)
-		)
-		(property "Voltage" "25V"
-			(at 138.43 102.87 0)
-			(hide yes)
-			(show_name no)
-			(do_not_autoplace no)
-			(effects
-				(font
-					(size 1.27 1.27)
-				)
-			)
-		)
 		(property "Mouser" "581-06033U100JAT2A"
 			(at 138.43 102.87 0)
@@
 		)
 		(property "LCSC" "C2229848"
+			(at 138.43 102.87 0)
+			(hide yes)
+			(show_name no)
+			(do_not_autoplace no)
+			(effects
+				(font
+					(size 1.27 1.27)
+				)
+			)
+		)
+		(property "Voltage_in_V" "25"
+			(at 138.43 102.87 0)
+			(hide yes)
+			(show_name no)
+			(do_not_autoplace no)
+			(effects
+				(font
+					(size 1.27 1.27)
+				)
+			)
+		)
+		(property "Tolerance_in_pct" "5"
+			(at 138.43 102.87 0)
+			(hide yes)
+			(show_name no)
+			(do_not_autoplace no)
+			(effects
+				(font
+					(size 1.27 1.27)
+				)
+			)
+		)
+		(property "Dielectric" "C0G"
+			(at 138.43 102.87 0)
+			(hide yes)
+			(show_name no)
+			(do_not_autoplace no)
+			(effects
+				(font
+					(size 1.27 1.27)
+				)
+			)
+		)
+		(property "Package_in_inch" "0603"
+			(at 138.43 102.87 0)
+			(hide yes)
+			(show_name no)
+			(do_not_autoplace no)
+			(effects
+				(font
+					(size 1.27 1.27)
+				)
+			)
+		)
+		(property "MPN" "06033U100JAT2A"
 			(at 138.43 102.87 0)
 			(hide yes)
@@
 	)
 	(symbol
-		(lib_id "KL_SYM_LOCAL:GND")
+		(lib_id "power:GND")
 		(at 149.86 95.25 0)
 		(unit 1)
@@
 	)
 	(symbol
-		(lib_id "KL_C:C_10p_25V_C0G_0603_5")
+		(lib_id "KL_C:C_10p_25V_5pct_C0G_0603")
 		(at 138.43 88.9 270)
 		(unit 1)
@@
 			)
 		)
-		(property "Datasheet" ""
+		(property "Datasheet" "https://datasheets.kyocera-avx.com/U-Series.pdf"
 			(at 138.43 88.9 0)
 			(hide yes)
@@
 			)
 		)
-		(property "Tolerance" "5"
-			(at 138.43 88.9 0)
-			(hide yes)
-			(show_name no)
-			(do_not_autoplace no)
-			(effects
-				(font
-					(size 1.27 1.27)
-				)
-			)
-		)
-		(property "Voltage" "25V"
-			(at 138.43 88.9 0)
-			(hide yes)
-			(show_name no)
-			(do_not_autoplace no)
-			(effects
-				(font
-					(size 1.27 1.27)
-				)
-			)
-		)
 		(property "Mouser" "581-06033U100JAT2A"
 			(at 138.43 88.9 0)
@@
 		)
 		(property "LCSC" "C2229848"
+			(at 138.43 88.9 0)
+			(hide yes)
+			(show_name no)
+			(do_not_autoplace no)
+			(effects
+				(font
+					(size 1.27 1.27)
+				)
+			)
+		)
+		(property "Voltage_in_V" "25"
+			(at 138.43 88.9 0)
+			(hide yes)
+			(show_name no)
+			(do_not_autoplace no)
+			(effects
+				(font
+					(size 1.27 1.27)
+				)
+			)
+		)
+		(property "Tolerance_in_pct" "5"
+			(at 138.43 88.9 0)
+			(hide yes)
+			(show_name no)
+			(do_not_autoplace no)
+			(effects
+				(font
+					(size 1.27 1.27)
+				)
+			)
+		)
+		(property "Dielectric" "C0G"
+			(at 138.43 88.9 0)
+			(hide yes)
+			(show_name no)
+			(do_not_autoplace no)
+			(effects
+				(font
+					(size 1.27 1.27)
+				)
+			)
+		)
+		(property "Package_in_inch" "0603"
+			(at 138.43 88.9 0)
+			(hide yes)
+			(show_name no)
+			(do_not_autoplace no)
+			(effects
+				(font
+					(size 1.27 1.27)
+				)
+			)
+		)
+		(property "MPN" "06033U100JAT2A"
 			(at 138.43 88.9 0)
 			(hide yes)
@@
 	)
 	(symbol
-		(lib_id "KL_Passive_ICs:Crystal_25MHz_32p")
+		(lib_id "KL_Crystal:Crystal_25M_10ppm_32pF_3.2x2.5")
 		(at 142.24 95.25 270)
 		(unit 1)
@@
 			)
 		)
-		(property "Value" "25000000"
+		(property "Value" "25M"
 			(at 159.766 61.722 0)
 			(hide yes)
@@
 			)
 		)
-		(property "Description" ""
+		(property "Description" "Crystal"
 			(at 142.24 95.25 0)
 			(hide yes)
@@
 			)
 		)
+		(property "Frequency_Tolerance_in_ppm" "10"
+			(at 142.24 95.25 0)
+			(hide yes)
+			(show_name no)
+			(do_not_autoplace no)
+			(effects
+				(font
+					(size 1.27 1.27)
+				)
+			)
+		)
+		(property "Load_Capacitance_in_pF" "32"
+			(at 142.24 95.25 0)
+			(hide yes)
+			(show_name no)
+			(do_not_autoplace no)
+			(effects
+				(font
+					(size 1.27 1.27)
+				)
+			)
+		)
+		(property "Package_LxW_in_mm" "3.2x2.5"
+			(at 142.24 95.25 0)
+			(hide yes)
+			(show_name no)
+			(do_not_autoplace no)
+			(effects
+				(font
+					(size 1.27 1.27)
+				)
+			)
+		)
+		(property "MPN" "VXM7-9032-25M0000000"
+			(at 142.24 95.25 0)
+			(hide yes)
+			(show_name no)
+			(do_not_autoplace no)
+			(effects
+				(font
+					(size 1.27 1.27)
+				)
+			)
+		)

Commit message: updates 10pF capacitor. Refs: #41
Parts:
- C86, C92: Digikey 06033U100JAT2A-ND -> 13-CC0603JRNPO8BN100CT-ND; LCSC C2229848 -> C1853175; MPN 06033U100JAT2A -> CC0603JRNPO8BN100; Mouser 581-06033U100JAT2A -> 603-CC0603JRNP8BN100
Changed lines of the file:
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@@
 		(fields_autoplaced yes)
 		(property "Reference" "C92"
-			(at 138.43 107.95 90)
+			(at 138.43 95.25 90)
 			(show_name no)
 			(do_not_autoplace no)
@@
 		)
 		(property "Value" "10p"
-			(at 138.43 110.49 90)
+			(at 138.43 97.79 90)
 			(show_name no)
 			(do_not_autoplace no)
@@
 			)
 		)
-		(property "Datasheet" "https://datasheets.kyocera-avx.com/U-Series.pdf"
+		(property "Datasheet" "https://yageogroup.com/download/specsheet/CC0603JRNPO8BN100"
 			(at 138.43 102.87 0)
 			(hide yes)
@@
 			)
 		)
-		(property "Mouser" "581-06033U100JAT2A"
-			(at 138.43 102.87 0)
-			(hide yes)
-			(show_name no)
-			(do_not_autoplace no)
-			(effects
-				(font
-					(size 1.27 1.27)
-				)
-			)
-		)
-		(property "Digikey" "06033U100JAT2A-ND"
-			(at 138.43 102.87 0)
-			(hide yes)
-			(show_name no)
-			(do_not_autoplace no)
-			(effects
-				(font
-					(size 1.27 1.27)
-				)
-			)
-		)
-		(property "LCSC" "C2229848"
+		(property "Mouser" "603-CC0603JRNP8BN100"
+			(at 138.43 102.87 0)
+			(hide yes)
+			(show_name no)
+			(do_not_autoplace no)
+			(effects
+				(font
+					(size 1.27 1.27)
+				)
+			)
+		)
+		(property "Digikey" "13-CC0603JRNPO8BN100CT-ND"
+			(at 138.43 102.87 0)
+			(hide yes)
+			(show_name no)
+			(do_not_autoplace no)
+			(effects
+				(font
+					(size 1.27 1.27)
+				)
+			)
+		)
+		(property "LCSC" "C1853175"
 			(at 138.43 102.87 0)
 			(hide yes)
@@
 			)
 		)
-		(property "MPN" "06033U100JAT2A"
+		(property "MPN" "CC0603JRNPO8BN100"
 			(at 138.43 102.87 0)
 			(hide yes)
@@
 			)
 		)
-		(property "Datasheet" "https://datasheets.kyocera-avx.com/U-Series.pdf"
+		(property "Datasheet" "https://yageogroup.com/download/specsheet/CC0603JRNPO8BN100"
 			(at 138.43 88.9 0)
 			(hide yes)
@@
 			)
 		)
-		(property "Mouser" "581-06033U100JAT2A"
-			(at 138.43 88.9 0)
-			(hide yes)
-			(show_name no)
-			(do_not_autoplace no)
-			(effects
-				(font
-					(size 1.27 1.27)
-				)
-			)
-		)
-		(property "Digikey" "06033U100JAT2A-ND"
-			(at 138.43 88.9 0)
-			(hide yes)
-			(show_name no)
-			(do_not_autoplace no)
-			(effects
-				(font
-					(size 1.27 1.27)
-				)
-			)
-		)
-		(property "LCSC" "C2229848"
+		(property "Mouser" "603-CC0603JRNP8BN100"
+			(at 138.43 88.9 0)
+			(hide yes)
+			(show_name no)
+			(do_not_autoplace no)
+			(effects
+				(font
+					(size 1.27 1.27)
+				)
+			)
+		)
+		(property "Digikey" "13-CC0603JRNPO8BN100CT-ND"
+			(at 138.43 88.9 0)
+			(hide yes)
+			(show_name no)
+			(do_not_autoplace no)
+			(effects
+				(font
+					(size 1.27 1.27)
+				)
+			)
+		)
+		(property "LCSC" "C1853175"
 			(at 138.43 88.9 0)
 			(hide yes)
@@
 			)
 		)
-		(property "MPN" "06033U100JAT2A"
-			(at 138.43 88.9 0)
-			(hide yes)
+		(property "MPN" "CC0603JRNPO8BN100"
+			(at 138.43 88.9 0)
+			(hide yes)
