File: buck_2v5.kicad_sch (KiCad schematic)
At the start: 20 parts, among them U3 TPS564257DRLR

Commit message: open project in KiCAD10. Refs: #41
Parts:
- TP28, TP29, TP30, TP31: value ~ -> (none)

Commit message: updates buck_2v5. Refs: #41
Parts:
- removed C98: 100n, KL_Footprints:C_0603, symbol KL_C:C_100n_10V_X7R_0603_10
- added C107: 100n, KL_Footprints:C_0603, symbol KL_C:C_100n_16V_10pct_X7R_0603
- C100, C101: value 10uF -> 10u; symbol KL_C:C_10u_25V_X5R_0603_20 -> KL_C:C_10u_25V_20pct_X5R_0603; Dielectric (none) -> X5R; MPN (none) -> CL10A106MA8NRNC; Package_in_inch (none) -> 0603; Tolerance 20 -> (none); Tolerance_in_pct (none) -> 20; Voltage 25 -> (none); Voltage_in_V (none) -> 25
- C102: symbol KL_C:C_100n_16V_X7R_0603_10 -> KL_C:C_100n_16V_10pct_X7R_0603; Dielectric (none) -> X7R; MPN (none) -> CC0603KPX7R7BB104; Package_in_inch (none) -> 0603; Tolerance 10 -> (none); Tolerance_in_pct (none) -> 10; Voltage 16V -> (none); Voltage_in_V (none) -> 16
- C103: symbol KL_C:C_10n_50V_X7R_0603_10 -> KL_C:C_10n_50V_10pct_X7R_0603; Dielectric (none) -> X7R; MPN (none) -> CL10B103KB8WPND; Package_in_inch (none) -> 0603; Tolerance 10 -> (none); Tolerance_in_pct (none) -> 10; Voltage 50 -> (none); Voltage_in_V (none) -> 50
- C96, C97: symbol KL_C:C_22u_10V_X5R_0603_20 -> KL_C:C_22u_10V_20pct_X5R_0603; Dielectric (none) -> X5R; MPN (none) -> GRM187R61A226ME15D; Package_in_inch (none) -> 0603; Tolerance 20 -> (none); Tolerance_in_pct (none) -> 20; Voltage 10V -> (none); Voltage_in_V (none) -> 10
- C99: symbol KL_C:C_10p_25V_C0G_0603_5 -> KL_C:C_10p_25V_5pct_C0G_0603; Dielectric (none) -> C0G; MPN (none) -> 06033U100JAT2A; Package_in_inch (none) -> 0603; Tolerance 5 -> (none); Tolerance_in_pct (none) -> 5; Voltage 25V -> (none); Voltage_in_V (none) -> 25
- D2: symbol KL_LED:LED_red_2V_0.03A -> KL_LED:LED_Red_2V_0.03A_0603; MPN (none) -> LTST-C194KRKT; Package_in_inch (none) -> 0603
- L3: symbol KL_L:L_3u3_8A_20pct_7LX7W -> KL_L:L_3u3_8A_20pct_7.2x6.9; MPN (none) -> EXLA1V0603-3R3-R; Package_LxW_in_mm (none) -> 7.2x6.9; Package_in_mm L7XW7 -> (none)
- R19: symbol KL_R:R_31K6_125mW_1_0603 -> KL_R:R_31K6_0.125W_1pct_0603; Farnell 2138454 -> (none); MPN (none) -> CRCW060331K6FKEA; Package (in) 0603 -> (none); Package_in_inch (none) -> 0603; Power 125mW -> (none); Power_in_W (none) -> 0.125; Tolerance 1% -> (none); Tolerance_in_pct (none) -> 1
- R85: symbol KL_R:R_10K_100mW_1_0603 -> KL_R:R_10K_0.1W_1pct_0603; Farnell 2421850 -> (none); MPN (none) -> RC0603FR-0710KL; Package (in) 0603 -> (none); Package_in_inch (none) -> 0603; Power_in_W (none) -> 0.1; Tolerance_in_pct (none) -> 1
- R95: symbol KL_R:R_1K5_100mW_5_0603 -> KL_R:R_1K5_0.1W_5pct_0603; MPN (none) -> AC0603JR-071K5L; Package (in) 0603 -> (none); Package_in_inch (none) -> 0603; Power 0.1 -> (none); Power_in_W (none) -> 0.1; Tolerance 5 -> (none); Tolerance_in_pct (none) -> 5
- R96: symbol KL_R:R_0R_2W_5_2512 -> KL_R:R_0R_2W_5pct_2512; MPN (none) -> CRF2512-J/-000ELF; Mouser 652-CRF2512-J-000ELF -> 652-CRF2512-J-000ELF; Package (in) 2512 -> (none); Package_in_inch (none) -> 2512; Power 2 -> (none); Power_in_W (none) -> 2; Tolerance 5 -> (none); Tolerance_in_pct (none) -> 5
- R99: symbol KL_R:R_10K_100mW_5_0603 -> KL_R:R_10K_0.1W_5pct_0603; MPN (none) -> CRCW060310K0JNEC; Package (in) 0603 -> (none); Package_in_inch (none) -> 0603; Power 100mW -> (none); Power_in_W (none) -> 0.1; Tolerance 5% -> (none); Tolerance_in_pct (none) -> 5
- TP28, TP29, TP30, TP31: footprint Connector_PinHeader_2.54mm:PinHeader_1x01_P2.54mm_Vertical -> KL_Footprints:TestPoint; symbol KL_TP:TestPoint -> KL_TestPoint:TestPoint
- U3: MPN (none) -> TPS564257DRLR; VIN_MAX_V (none) -> 17; VIN_MIN_V (none) -> 3
Connections:
- net +2V5_OUT: now also C107.1
- net GND: now also C107.2

Commit message: updates 10pF capacitor. Refs: #41
Parts:
- C99: Digikey 06033U100JAT2A-ND -> 13-CC0603JRNPO8BN100CT-ND; LCSC C2229848 -> C1853175; MPN 06033U100JAT2A -> CC0603JRNPO8BN100; Mouser 581-06033U100JAT2A -> 603-CC0603JRNP8BN100
Changed lines of the file:
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@@
 			)
 		)
-		(property "Datasheet" "https://datasheets.kyocera-avx.com/U-Series.pdf"
+		(property "Datasheet" "https://yageogroup.com/download/specsheet/CC0603JRNPO8BN100"
 			(at 173.99 83.82 0)
 			(hide yes)
@@
 			)
 		)
-		(property "Mouser" "581-06033U100JAT2A"
+		(property "Mouser" "603-CC0603JRNP8BN100"
 			(at 173.99 83.82 0)
 			(hide yes)
@@
 			)
 		)
-		(property "Digikey" "06033U100JAT2A-ND"
+		(property "Digikey" "13-CC0603JRNPO8BN100CT-ND"
 			(at 173.99 83.82 0)
 			(hide yes)
@@
 			)
 		)
-		(property "LCSC" "C2229848"
+		(property "LCSC" "C1853175"
 			(at 173.99 83.82 0)
 			(hide yes)
@@
 			)
 		)
-		(property "MPN" "06033U100JAT2A"
+		(property "MPN" "CC0603JRNPO8BN100"
 			(at 173.99 83.82 0)
 			(hide yes)

Commit message: replaces all capacitors with 10u. Refs: #52
Parts:
- C102, C107: value 100n -> 10u; symbol KL_C:C_100n_16V_10pct_X7R_0603 -> KL_C:C_10u_25V_20pct_X5R_0603; Dielectric X7R -> X5R; Digikey 311-1335-1-ND -> 1276-1869-1-ND; LCSC C2649559 -> C96446; MPN CC0603KPX7R7BB104 -> CL10A106MA8NRNC; Mouser 603-C0603KPX7R7BB104 -> 187-CL10A106MA8NRNC; Tolerance_in_pct 10 -> 20; Voltage_in_V 16 -> 25
- C96, C97: value 22u -> 10u; symbol KL_C:C_22u_10V_20pct_X5R_0603 -> KL_C:C_10u_25V_20pct_X5R_0603; Digikey 490-13243-1-ND -> 1276-1869-1-ND; LCSC C361061 -> C96446; MPN GRM187R61A226ME15D -> CL10A106MA8NRNC; Mouser 81-GRM187R61A226ME5D -> 187-CL10A106MA8NRNC; Voltage_in_V 10 -> 25
Changed lines of the file:
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@@
 	)
 	(symbol
-		(lib_id "KL_C:C_100n_16V_10pct_X7R_0603")
+		(lib_id "KL_C:C_10u_25V_20pct_X5R_0603")
 		(at 99.06 88.9 0)
 		(unit 1)
@@
 			)
 		)
-		(property "Value" "100n"
+		(property "Value" "10u"
 			(at 102.87 90.1699 0)
 			(show_name no)
@@
 			)
 		)
-		(property "Datasheet" "https://yageogroup.com/download/specsheet/CC0603KPX7R7BB104"
+		(property "Datasheet" "https://weblib.samsungsem.com/mlcc/mlcc-ec-data-sheet.do?partNumber=CL10A106MA8NRN"
 			(at 99.06 88.9 0)
 			(hide yes)
@@
 			)
 		)
-		(property "Mouser" "603-C0603KPX7R7BB104"
+		(property "Mouser" "187-CL10A106MA8NRNC"
 			(at 99.06 88.9 0)
 			(hide yes)
@@
 			)
 		)
-		(property "Digikey" "311-1335-1-ND"
+		(property "Digikey" "1276-1869-1-ND"
 			(at 99.06 88.9 0)
 			(hide yes)
@@
 			)
 		)
-		(property "LCSC" "C2649559"
+		(property "LCSC" "C96446"
 			(at 99.06 88.9 0)
 			(hide yes)
@@
 			)
 		)
-		(property "Voltage_in_V" "16"
+		(property "Voltage_in_V" "25"
 			(at 99.06 88.9 0)
 			(hide yes)
@@
 			)
 		)
-		(property "Tolerance_in_pct" "10"
+		(property "Tolerance_in_pct" "20"
 			(at 99.06 88.9 0)
 			(hide yes)
@@
 			)
 		)
-		(property "Dielectric" "X7R"
+		(property "Dielectric" "X5R"
 			(at 99.06 88.9 0)
 			(hide yes)
@@
 			)
 		)
-		(property "MPN" "CC0603KPX7R7BB104"
+		(property "MPN" "CL10A106MA8NRNC"
 			(at 99.06 88.9 0)
 			(hide yes)
@@
 	)
 	(symbol
-		(lib_id "KL_C:C_100n_16V_10pct_X7R_0603")
+		(lib_id "KL_C:C_10u_25V_20pct_X5R_0603")
 		(at 234.95 82.55 0)
 		(unit 1)
@@
 			)
 		)
-		(property "Value" "100n"
+		(property "Value" "10u"
 			(at 238.76 83.8199 0)
 			(show_name no)
@@
 			)
 		)
-		(property "Datasheet" "https://yageogroup.com/download/specsheet/CC0603KPX7R7BB104"
+		(property "Datasheet" "https://weblib.samsungsem.com/mlcc/mlcc-ec-data-sheet.do?partNumber=CL10A106MA8NRN"
 			(at 234.95 82.55 0)
 			(hide yes)
@@
 			)
 		)
-		(property "Mouser" "603-C0603KPX7R7BB104"
+		(property "Mouser" "187-CL10A106MA8NRNC"
 			(at 234.95 82.55 0)
 			(hide yes)
@@
 			)
 		)
-		(property "Digikey" "311-1335-1-ND"
+		(property "Digikey" "1276-1869-1-ND"
 			(at 234.95 82.55 0)
 			(hide yes)
@@
 			)
 		)
-		(property "LCSC" "C2649559"
+		(property "LCSC" "C96446"
 			(at 234.95 82.55 0)
 			(hide yes)
@@
 			)
 		)
-		(property "Voltage_in_V" "16"
+		(property "Voltage_in_V" "25"
 			(at 234.95 82.55 0)
 			(hide yes)
@@
 			)
 		)
-		(property "Tolerance_in_pct" "10"
+		(property "Tolerance_in_pct" "20"
 			(at 234.95 82.55 0)
 			(hide yes)
@@
 			)
 		)
-		(property "Dielectric" "X7R"
+		(property "Dielectric" "X5R"
 			(at 234.95 82.55 0)
 			(hide yes)
@@
 			)
 		)
-		(property "MPN" "CC0603KPX7R7BB104"
+		(property "MPN" "CL10A106MA8NRNC"
 			(at 234.95 82.55 0)
 			(hide yes)
@@
 	)
 	(symbol
-		(lib_id "KL_C:C_22u_10V_20pct_X5R_0603")
+		(lib_id "KL_C:C_10u_25V_20pct_X5R_0603")
 		(at 212.09 82.55 0)
 		(unit 1)
@@
 			)
 		)
-		(property "Value" "22u"
+		(property "Value" "10u"
 			(at 215.9 83.8199 0)
 			(show_name no)
@@
 			)
 		)
-		(property "Datasheet" "https://pim.murata.com/asset/pim4/ceramicCapacitorSMD/GRM187R61A226ME15-01A-EN_PDF_CERAMICCAPACITORSMD"
+		(property "Datasheet" "https://weblib.samsungsem.com/mlcc/mlcc-ec-data-sheet.do?partNumber=CL10A106MA8NRN"
 			(at 212.09 82.55 0)
 			(hide yes)
@@
 			)
 		)
-		(property "Mouser" "81-GRM187R61A226ME5D"
+		(property "Mouser" "187-CL10A106MA8NRNC"
 			(at 212.09 82.55 0)
 			(hide yes)
@@
 			)
 		)
-		(property "Digikey" "490-13243-1-ND"
+		(property "Digikey" "1276-1869-1-ND"
 			(at 212.09 82.55 0)
 			(hide yes)
@@
 			)
 		)
-		(property "LCSC" "C361061"
+		(property "LCSC" "C96446"
 			(at 212.09 82.55 0)
 			(hide yes)
@@
 			)
 		)
-		(property "Voltage_in_V" "10"
+		(property "Voltage_in_V" "25"
 			(at 212.09 82.55 0)
 			(hide yes)
@@
 			)
 		)
-		(property "MPN" "GRM187R61A226ME15D"
+		(property "MPN" "CL10A106MA8NRNC"
 			(at 212.09 82.55 0)
 			(hide yes)
@@
 	)
 	(symbol
-		(lib_id "KL_C:C_22u_10V_20pct_X5R_0603")
+		(lib_id "KL_C:C_10u_25V_20pct_X5R_0603")
 		(at 223.52 82.55 0)
 		(unit 1)
@@
 			)
 		)
-		(property "Value" "22u"
+		(property "Value" "10u"
 			(at 227.33 83.8199 0)
 			(show_name no)
@@
 			)
 		)
-		(property "Datasheet" "https://pim.murata.com/asset/pim4/ceramicCapacitorSMD/GRM187R61A226ME15-01A-EN_PDF_CERAMICCAPACITORSMD"
+		(property "Datasheet" "https://weblib.samsungsem.com/mlcc/mlcc-ec-data-sheet.do?partNumber=CL10A106MA8NRN"
 			(at 223.52 82.55 0)
 			(hide yes)
@@
 			)
 		)
-		(property "Mouser" "81-GRM187R61A226ME5D"
+		(property "Mouser" "187-CL10A106MA8NRNC"
 			(at 223.52 82.55 0)
 			(hide yes)
@@
 			)
 		)
-		(property "Digikey" "490-13243-1-ND"
+		(property "Digikey" "1276-1869-1-ND"
 			(at 223.52 82.55 0)
 			(hide yes)
@@
 			)
 		)
-		(property "LCSC" "C361061"
+		(property "LCSC" "C96446"
 			(at 223.52 82.55 0)
 			(hide yes)
@@
 			)
 		)
-		(property "Voltage_in_V" "10"
+		(property "Voltage_in_V" "25"
 			(at 223.52 82.55 0)
 			(hide yes)
@@
 			)
 		)
-		(property "MPN" "GRM187R61A226ME15D"
+		(property "MPN" "CL10A106MA8NRNC"
 			(at 223.52 82.55 0)
 			(hide yes)
