File: switch_power_buffer_caps.kicad_sch (KiCad schematic)
At the start: 44 parts

Commit message: updates component details for ordering. Refs: #1
Parts:
- C25, C35, C38: Mouser 80-C0603C475K8PAC -> 80-C0603C475K8PACLR

Commit message: updates switch_power_buffer_caps. Refs:#41
Parts:
- C25, C35, C38: symbol KL_C:C_4u7_10V_X5R_0603_10 -> KL_C:C_4u7_10V_10pct_X5R_0603; Dielectric (none) -> X5R; MPN (none) -> C0603C475K8PAC7411; Package_in_inch (none) -> 0603; Tolerance 10 -> (none); Tolerance_in_pct (none) -> 10; Voltage 10 -> (none); Voltage_in_V (none) -> 10
- C27, C28, C29, C30, C31, C32, C33, C34, C36, C37, C39, C40, C41, C42, C43, C44, C45, C46, C47, C48, C49, C50, C51, C52, C53, C54, C55, C56, C57, C58, C59, C60, C61, C62, C63, C64, C65, C66, C67, C68, C69: symbol KL_C:C_100n_16V_X7R_0603_10 -> KL_C:C_100n_16V_10pct_X7R_0603; Dielectric (none) -> X7R; MPN (none) -> CC0603KPX7R7BB104; Package_in_inch (none) -> 0603; Tolerance 10 -> (none); Tolerance_in_pct (none) -> 10; Voltage 16V -> (none); Voltage_in_V (none) -> 16

Commit message: replaces all capacitors with 10u. Refs: #52
Parts:
- C25, C35, C38: value 4u7 -> 10u; symbol KL_C:C_4u7_10V_10pct_X5R_0603 -> KL_C:C_10u_25V_20pct_X5R_0603; Digikey 399-C0603C475K8PACTUCT-ND -> 1276-1869-1-ND; LCSC C5177163 -> C96446; MPN C0603C475K8PAC7411 -> CL10A106MA8NRNC; Mouser 80-C0603C475K8PACLR -> 187-CL10A106MA8NRNC; Tolerance_in_pct 10 -> 20; Voltage_in_V 10 -> 25
- C27, C28, C29, C30, C31, C32, C33, C34, C36, C37, C39, C40, C41, C42, C43, C44, C45, C46, C47, C48, C49, C50, C51, C52, C53, C54, C55, C56, C57, C58, C59, C60, C61, C62, C63, C64, C65, C66, C67, C68, C69: value 100n -> 10u; symbol KL_C:C_100n_16V_10pct_X7R_0603 -> KL_C:C_10u_25V_20pct_X5R_0603; Dielectric X7R -> X5R; Digikey 311-1335-1-ND -> 1276-1869-1-ND; LCSC C2649559 -> C96446; MPN CC0603KPX7R7BB104 -> CL10A106MA8NRNC; Mouser 603-C0603KPX7R7BB104 -> 187-CL10A106MA8NRNC; Tolerance_in_pct 10 -> 20; Voltage_in_V 16 -> 25
