File: shish-lan.kicad_pcb (KiCad board)
At the start: 2 copper layers, 309 parts, among them J1 0826-1X4T-43-F, J10 07x01_2.54mm_Header, J11 02x10_2.54mm_Header_Odd_Even, J2 02x01_2.54mm_Header, J3 02x01_2.54mm_Header, J4 03x01_2.54mm_Header, J5 02x10_2.54mm_Header_Odd_Even, J6 03x01_2.54mm_Header, J7 03x01_2.54mm_Header, J8 02x01_2.54mm_Header, J9 07x01_2.54mm_Header, U1 LAN96455F-I/8MW, U2 TPS564257DRLR, U3 TPS564257DRLR, U4 STM32H742VGT6, U5 TPS564257DRLR, X1 25000000, X2 25000000

Commit message: initial commit for RJ45 header, mounting holes, power connectors, PPS, GND TP. Refs: #43
Parts:
- removed C74: 100n, KL_Footprints:C_0603
- removed R24, R86, R90, R91: 0R, KL_Footprints:R_2512
- added C107: 100n, KL_Footprints:C_0603, F.Cu at (395.9, 21.3)
- added G***: LOGO, LOGO, F.Cu at (63.5, 29.5)
- added J13: SMA, KL_Footprints:SMA_Right_Angle, F.Cu at (369.6, 65.6)
- added J14: SMA, KL_Footprints:SMA_Right_Angle, F.Cu at (63.0, 120.0)
- added R98: 0R, KL_Footprints:R_0603, F.Cu at (354.5, 64.3)
- C1, C18, C19, C20, C21: footprint KL_Footprints:C_0603 -> KL_Footprints:C_0402
- C100, C101, C75, C76, C88, C89: value 10uF -> 10u
- FB1, FB2, FB3, FB4, FB5: footprint KL_Footprints:BLM18P -> KL_Footprints:FB_0603
- J1: value 0826-1X4T-43-F -> RJ45_0826-1X4T-43-F
- J10, J9: value 07x01_2.54mm_Header -> Header_07x01_2.54mm_0mm_Straight
- J11, J5: value 02x10_2.54mm_Header_Odd_Even -> Header_10x02_2.54mm_2.54mm_Straight
- J2, J3, J8: value 02x01_2.54mm_Header -> Header_02x01_2.54mm_0mm_Straight
- J4, J6, J7: value 03x01_2.54mm_Header -> Header_03x01_2.54mm_0mm_Straight
- R110, R111, R113, R114, R115, R116, R117, R118, R74: value 22 -> 22R
- R112: footprint KL_Footprints:R_2512 -> KL_Footprints:R_0603
- R71: value 10K -> 10R
- R75, R76, R77, R78: value 330 -> 330R
- TP1, TP10, TP11, TP12, TP13, TP14, TP15, TP16, TP17, TP18, TP19, TP2, TP20, TP21, TP22, TP23, TP24, TP25, TP26, TP27, TP28, TP29, TP3, TP30, TP31, TP32, TP33, TP34, TP35, TP4, TP5, TP6, TP7, TP8, TP9: footprint Connector_PinHeader_2.54mm:PinHeader_1x01_P2.54mm_Vertical -> KL_Footprints:TestPoint
- U4: footprint Package_QFP:LQFP-100_14x14mm_P0.5mm -> KL_Footprints:LQFP-100_14x14mm_P0.5mm
- X1, X2: value 25000000 -> 25M
- moved C21 339.7 mm to (404.9, 78.6)
- moved C20 339.7 mm to (404.9, 76.7)
- moved C19 339.7 mm to (404.9, 74.7)
- moved C18 339.7 mm to (404.9, 72.7)
- moved C1 339.6 mm to (404.9, 70.7)
- moved R120 336.7 mm to (391.0, 77.1)
- moved R121 336.7 mm to (391.0, 82.0)
- moved FB5 336.5 mm to (397.4, 81.2)
- moved FB4 336.4 mm to (397.4, 78.7)
- moved FB3 336.3 mm to (397.4, 76.1)
- moved FB2 336.3 mm to (397.4, 73.6)
- moved FB1 336.2 mm to (397.4, 71.0)
- moved R88 336.2 mm to (391.0, 72.2)
- moved C106 332.2 mm to (401.4, 71.0)
- moved R71 332.2 mm to (401.4, 73.5)
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Connections:
- C1 pad 1: Net-(C1-Pad1) -> /switch/2V5_BUCK-OUT
- C18 pad 1: Net-(C18-Pad1) -> /switch/2V5_BUCK-OUT
- C19 pad 1: Net-(C19-Pad1) -> /switch/1V15_BUCK-OUT
- C20 pad 1: Net-(C20-Pad1) -> /switch/1V15_BUCK-OUT
- C98 pad 1: /switch/2V5_BUCK-OUT -> +3V3
- FB2 pad 1: Net-(C20-Pad1) -> /switch/1V15_BUCK-OUT
- FB3 pad 1: Net-(C19-Pad1) -> /switch/1V15_BUCK-OUT
- FB4 pad 1: Net-(C18-Pad1) -> /switch/2V5_BUCK-OUT
- FB5 pad 1: Net-(C1-Pad1) -> /switch/2V5_BUCK-OUT
Other:
- board outline added: 100 x 100 mm

Commit message: shish-lan: pbc: adding proposition, movin sma and moving power, adding header as well
Parts:
- moved J11 282.5 mm to (58.5, 50.0)
- moved J5 277.8 mm to (61.0, 107.4), turned to 180 degrees
- moved G*** 93.0 mm to (83.3, 120.4)
- moved J14 90.1 mm to (68.5, 30.0), turned to 180 degrees
- moved J8 40.5 mm to (96.6, 95.7)
- moved J12 35.8 mm to (99.2, 124.0)
- moved J1 9.43 mm to (109.4, 25.7)
- moved TP13 1.30 mm to (53.0, 114.5)

Commit message: layout v1
Parts:
- removed C24: 100n, KL_Footprints:C_0603
- removed R111: 22R, KL_Footprints:R_0603
- removed R16, R96: 0R, KL_Footprints:R_2512
- removed R75, R76, R77, R78: 330R, KL_Footprints:R_0603
- added C108: 10u, KL_Footprints:C_0603, F.Cu at (99.4, 104.1)
- added C109: 10u, KL_Footprints:C_0603, F.Cu at (120.2, 104.1)
- added C74: 10u, KL_Footprints:C_0603, F.Cu at (78.6, 104.1)
- added J15: Header_02x01_2.54mm_0mm_Straight, KL_Footprints:02x01_2.54mm_Header, F.Cu at (115.6, 104.3)
- added J16: Header_02x01_2.54mm_0mm_Straight, KL_Footprints:02x01_2.54mm_Header, F.Cu at (73.8, 104.2)
- added J17: Header_02x01_2.54mm_0mm_Straight, KL_Footprints:02x01_2.54mm_Header, F.Cu at (94.8, 104.2)
- C1, C18, C19, C20, C21: footprint KL_Footprints:C_0402 -> KL_Footprints:C_0603
- C102, C104, C107, C27, C28, C29, C30, C31, C32, C33, C34, C36, C37, C39, C40, C41, C42, C43, C44, C45, C46, C47, C48, C49, C50, C51, C52, C53, C54, C55, C56, C57, C58, C59, C60, C61, C62, C63, C64, C65, C66, C67, C68, C69, C72, C77, C78, C79, C85, C90, C93, C94, C95, C98: value 100n -> 10u
- C105, C25, C35, C38: value 4u7 -> 10u
- C26, C70, C71, C73, C96, C97: value 22u -> 10u
- moved R8 359.9 mm to (56.3, 45.2)
- moved R4 358.9 mm to (56.3, 46.8), turned to 180 degrees
- moved C12 357.5 mm to (56.3, 43.6)
- moved C11 357.3 mm to (56.3, 42.0), turned to 180 degrees
- moved R2 355.0 mm to (56.3, 38.7)
- moved C9 353.6 mm to (56.3, 37.1)
- moved C10 353.4 mm to (56.3, 40.4)
- moved C80 342.1 mm to (62.6, 112.6), turned to 90 degrees
- moved R82 339.3 mm to (65.1, 118.2)
- moved D3 338.4 mm to (66.5, 108.7), turned to 90 degrees
- moved TP8 338.4 mm to (60.9, 91.4)
- moved R84 338.3 mm to (64.4, 112.6), turned to 90 degrees
- moved C19 336.9 mm to (68.9, 100.0)
- moved R79 336.4 mm to (68.6, 118.2)
- moved C62 336.2 mm to (53.2, 67.7)
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Connections:
- C1 pad 1: /switch/2V5_BUCK-OUT -> /switch/switch_power/2V5_PWR_SWITCH
- C100 pad 1: Net-(U3-VIN) -> /5-12V_INPUT
- C101 pad 1: Net-(U3-VIN) -> /5-12V_INPUT
- C102 pad 1: Net-(U3-VIN) -> /5-12V_INPUT
- C104 pad 1: +3V3 -> /controller/VDD_CTRL
- C105 pad 1: +3V3 -> /controller/VDD_CTRL
- C18 pad 1: /switch/2V5_BUCK-OUT -> /switch/switch_power/2V5_PWR_SWITCH
- C19 pad 1: /switch/1V15_BUCK-OUT -> /switch/switch_power/1V15_PWR_SWITCH
- C20 pad 1: /switch/1V15_BUCK-OUT -> /switch/switch_power/1V15_PWR_SWITCH
- C25 pad 1: /switch/1V15_BUCK-OUT -> /switch/switch_power/1V15_PWR_SWITCH
- C41 pad 1: /switch/1V15_BUCK-OUT -> /switch/switch_power/1V15_PWR_SWITCH
- C42 pad 1: /switch/1V15_BUCK-OUT -> /switch/switch_power/1V15_PWR_SWITCH
- C43 pad 1: /switch/1V15_BUCK-OUT -> /switch/switch_power/1V15_PWR_SWITCH
- C44 pad 1: /switch/1V15_BUCK-OUT -> /switch/switch_power/1V15_PWR_SWITCH
- C45 pad 1: /switch/1V15_BUCK-OUT -> /switch/switch_power/1V15_PWR_SWITCH
- C46 pad 1: /switch/1V15_BUCK-OUT -> /switch/switch_power/1V15_PWR_SWITCH
- C47 pad 1: /switch/1V15_BUCK-OUT -> /switch/switch_power/1V15_PWR_SWITCH
- C48 pad 1: /switch/1V15_BUCK-OUT -> /switch/switch_power/1V15_PWR_SWITCH
- C49 pad 1: /switch/1V15_BUCK-OUT -> /switch/switch_power/1V15_PWR_SWITCH
- C50 pad 1: /switch/1V15_BUCK-OUT -> /switch/switch_power/1V15_PWR_SWITCH
- C51 pad 1: /switch/1V15_BUCK-OUT -> /switch/switch_power/1V15_PWR_SWITCH
- C52 pad 1: /switch/1V15_BUCK-OUT -> /switch/switch_power/1V15_PWR_SWITCH
- C53 pad 1: /switch/1V15_BUCK-OUT -> /switch/switch_power/1V15_PWR_SWITCH
- C54 pad 1: /switch/1V15_BUCK-OUT -> /switch/switch_power/1V15_PWR_SWITCH
- C55 pad 1: /switch/1V15_BUCK-OUT -> /switch/switch_power/1V15_PWR_SWITCH
- C56 pad 1: /switch/1V15_BUCK-OUT -> /switch/switch_power/1V15_PWR_SWITCH
- C57 pad 1: /switch/1V15_BUCK-OUT -> /switch/switch_power/1V15_PWR_SWITCH
- C75 pad 1: Net-(U2-VIN) -> /5-12V_INPUT
- C76 pad 1: Net-(U2-VIN) -> /5-12V_INPUT
- C77 pad 1: +3V3 -> /controller/VDD_CTRL
- C78 pad 1: +3V3 -> /controller/VDD_CTRL
- C79 pad 1: Net-(U2-VIN) -> /5-12V_INPUT
- C85 pad 1: +3V3 -> /controller/VDD_CTRL
- C87 pad 1: +3V3 -> Net-(J15-Pin_2)
- C93 pad 1: +3V3 -> /controller/VDD_CTRL
- C94 pad 1: +3V3 -> /controller/VDD_CTRL
- C95 pad 1: +3V3 -> /controller/VDD_CTRL
- C99 pad 1: /switch/2V5_BUCK-OUT -> Net-(J17-Pin_2)
- D4 pad 2: +3V3 -> /controller/VDD_CTRL
- D5 pad 2: +3V3 -> /controller/VDD_CTRL
- D6 pad 2: +3V3 -> /controller/VDD_CTRL
- FB1 pad 1: /switch/1V15_BUCK-OUT -> /switch/switch_power/1V15_PWR_SWITCH
- FB2 pad 1: /switch/1V15_BUCK-OUT -> /switch/switch_power/1V15_PWR_SWITCH
- FB3 pad 1: /switch/1V15_BUCK-OUT -> /switch/switch_power/1V15_PWR_SWITCH
- FB4 pad 1: /switch/2V5_BUCK-OUT -> /switch/switch_power/2V5_PWR_SWITCH
- FB5 pad 1: /switch/2V5_BUCK-OUT -> /switch/switch_power/2V5_PWR_SWITCH
- J1 pad S1: Net-(J1A-SHIELD) -> GND
- J1 pad S2: Net-(J1A-SHIELD__1) -> GND
- J1 pad S3: Net-(J1A-SHIELD__2) -> GND
- J1 pad S4: Net-(J1A-SHIELD__3) -> GND
- J9 pad 2: /controller/RGMII0_SWITCH_STM.TXCTL-DX_DV -> /controller/RGMII0_SWITCH_STM.TXD3
- J9 pad 3: /controller/RGMII0_SWITCH_STM.TXC-REFCLK -> /controller/RGMII0_SWITCH_STM.TXD2
- J9 pad 4: /controller/RGMII0_SWITCH_STM.TXD3 -> /controller/RGMII0_SWITCH_STM.TXD1
- J9 pad 5: /controller/RGMII0_SWITCH_STM.TXD2 -> /controller/RGMII0_SWITCH_STM.TXD0
- J9 pad 6: /controller/RGMII0_SWITCH_STM.TXD1 -> /controller/RGMII0_SWITCH_STM.TXCTL-DX_DV
- J9 pad 7: /controller/RGMII0_SWITCH_STM.TXD0 -> /controller/RGMII0_SWITCH_STM.TXC-REFCLK
- L1 pad 2: +3V3 -> Net-(J15-Pin_2)
- L2 pad 2: /switch/1V15_BUCK-OUT -> Net-(J16-Pin_2)
- L3 pad 2: /switch/2V5_BUCK-OUT -> Net-(J17-Pin_2)
- R102 pad 1: +3V3 -> /controller/VDD_CTRL
- R108 pad 2: Net-(U4-VBAT) -> /controller/VDD_CTRL
- R109 pad 2: +3V3 -> /controller/VDD_CTRL
- R120 pad 2: /switch/2V5_BUCK-OUT -> /switch/switch_power/2V5_PWR_SWITCH
- R121 pad 2: /switch/1V15_BUCK-OUT -> /switch/switch_power/1V15_PWR_SWITCH
- R19 pad 1: /switch/2V5_BUCK-OUT -> Net-(J17-Pin_2)
- R20 pad 1: +3V3 -> Net-(J15-Pin_2)
- R80 pad 1: +3V3 -> Net-(J15-Pin_2)
- R82 pad 1: /switch/1V15_BUCK-OUT -> Net-(J16-Pin_2)
- R97 pad 2: +3V3 -> /controller/VDD_CTRL
- TP29 pad 1: Net-(U3-VIN) -> /5-12V_INPUT
- TP3 pad 1: Net-(U2-VIN) -> /5-12V_INPUT
- TP8 pad 1: /switch/1V15_BUCK-OUT -> /switch/switch_power/1V15_PWR_SWITCH
- U1 pad 122: /switch/1V15_BUCK-OUT -> /switch/switch_power/1V15_PWR_SWITCH
- U1 pad 37: /switch/1V15_BUCK-OUT -> /switch/switch_power/1V15_PWR_SWITCH
- U1 pad 59: /switch/1V15_BUCK-OUT -> /switch/switch_power/1V15_PWR_SWITCH
- U1 pad 73: /switch/1V15_BUCK-OUT -> /switch/switch_power/1V15_PWR_SWITCH
- U1 pad 88: /switch/1V15_BUCK-OUT -> /switch/switch_power/1V15_PWR_SWITCH
- U2 pad 1: Net-(U2-VIN) -> /5-12V_INPUT
- U3 pad 1: Net-(U3-VIN) -> /5-12V_INPUT
- U4 pad 100: Net-(U4-VBAT) -> /controller/VDD_CTRL
- U4 pad 11: Net-(U4-VBAT) -> /controller/VDD_CTRL
- U4 pad 20: +3V3 -> /controller/VDD_CTRL
- U4 pad 21: Net-(U4-VBAT) -> /controller/VDD_CTRL
- U4 pad 27: Net-(U4-VBAT) -> /controller/VDD_CTRL
- U4 pad 47: Net-(U4-PB11) -> /controller/RGMII0_SWITCH_STM.TXCTL-DX_DV
- U4 pad 50: Net-(U4-VBAT) -> /controller/VDD_CTRL
- U4 pad 6: Net-(U4-VBAT) -> /controller/VDD_CTRL
- U4 pad 75: Net-(U4-VBAT) -> /controller/VDD_CTRL
Routing:
- net /switch/EN-1V15_STM_TO_BUCK: track 0.00 -> 117.7 mm, vias 0 -> 3
- net /5-12V_INPUT: track 0.00 -> 99.7 mm
- net /switch/IRQ0_SWITCH_TO_STM: track 0.00 -> 90.8 mm, vias 0 -> 4
- net /switch/EN-2V5_STM_TO_BUCK: track 0.00 -> 88.1 mm, vias 0 -> 4
- net /switch/nRST_STM_TO_SWITCH: track 0.00 -> 76.9 mm, vias 0 -> 4
- net /controller/SPI2_STM_SWITCH.nCS: track 0.00 -> 72.3 mm, vias 0 -> 4
- net /controller/debug_header/P1: track 0.00 -> 63.0 mm, vias 0 -> 2
- net /controller/VDD_CTRL: track 0.00 -> 61.1 mm, vias 0 -> 25
- net /controller/SPI2_STM_SWITCH.MOSI: track 0.00 -> 59.1 mm, vias 0 -> 3
- net /controller/SPI2_STM_SWITCH.CLK: track 0.00 -> 58.2 mm, vias 0 -> 5
- net /controller/debug_header/P9: track 0.00 -> 57.4 mm, vias 0 -> 2
- net /controller/debug_header/P2: track 0.00 -> 57.1 mm, vias 0 -> 2
- net /controller/RGMII0_SWITCH_STM.RXD1: track 0.00 -> 56.8 mm, vias 0 -> 2
- net /controller/debug_header/P11: track 0.00 -> 56.2 mm, vias 0 -> 2
- net /switch/switch_gpios/PHY0_LED1: track 0.00 -> 55.7 mm, vias 0 -> 1
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- added copper zone on In2.Cu, net +3V3
- added copper zone on In2.Cu, net /controller/VDD_CTRL
- added copper zone on F.Cu, net /switch/1V15_BUCK-OUT
- added copper zone on F.Cu, net /switch/2V5_BUCK-OUT
- added copper zone on In2.Cu, net /switch/switch_power/1V15_PWR_SWITCH
- added copper zone on In3.Cu, net /switch/switch_power/VDDIO
- added copper zone on B.Cu, net /switch/switch_power/VDDIO_PHY_AH
- added copper zone on In3.Cu, net /switch/switch_power/VDD_PHYS
- added copper zone on F.Cu, net GND
- added copper zone on In1.Cu, net GND
- added copper zone on In3.Cu, net GND
- added copper zone on In4.Cu, net GND
- added copper zone on F.Cu, net Net-(J15-Pin_2)
- added copper zone on F.Cu, net Net-(J16-Pin_2)
- added copper zone on F.Cu, net Net-(J17-Pin_2)
- added copper zone on F.Cu, net Net-(U2-SW)
- added copper zone on F.Cu, net Net-(U3-SW)
- added copper zone on F.Cu, net Net-(U5-SW)
Other:
- copper layers 2 -> 6
- board text added: "⏚"
