File: shish-lan.kicad_pcb (KiCad board)
At the start: 6 copper layers, 100 x 100 mm, 307 parts, among them J1 RJ45_0826-1X4T-43-F, J10 Header_07x01_2.54mm_0mm_Strai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, J11 Header_10x02_2.54mm_2.54mm_St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, J13 SMA, J14 SMA, J15 Header_02x01_2.54mm_0mm_Strai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, J16 Header_02x01_2.54mm_0mm_Strai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, J17 Header_02x01_2.54mm_0mm_Strai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, J2 Header_02x01_2.54mm_0mm_Strai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, J3 Header_02x01_2.54mm_0mm_Strai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, J4 Header_03x01_2.54mm_0mm_Strai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, J5 Header_10x02_2.54mm_2.54mm_St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, J6 Header_03x01_2.54mm_0mm_Strai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, J7 Header_03x01_2.54mm_0mm_Strai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, J8 Header_02x01_2.54mm_0mm_Strai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, J9 Header_07x01_2.54mm_0mm_Strai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, U1 LAN96455F-I/8MW, U2 TPS564257DRLR, U3 TPS564257DRLR, U4 STM32H742VGT6, U5 TPS564257DRLR, X1 25M, X2 25M

Commit message: Refs: 108 preparing the pcb for next revision B
Parts:
- removed J6: Header_03x01_2.54mm_0mm_Straight, KL_Footprints:03x01_2.54mm_Header
- removed TP23, TP32: ~, KL_Footprints:TestPoint
- added R138: 22R, KL_Footprints:R_0603, F.Cu at (123.0, 89.5)
- R133: value 0R -> 10K
- R69: value 10K -> 1K5
- moved R102 4.87 mm to (147.3, 92.5)
- moved G*** 2.31 mm to (56.0, 62.2)
- moved C81 0.11 mm to (123.3, 91.1)
Connections:
- net /switch/switch_gpios/JTAG_EN renamed /switch/switch_gpios/JTAG_ENB
- C103 pad 1: /switch/EN-2V5_STM_TO_BUCK -> +3V3
- C80 pad 1: /switch/EN-1V15_STM_TO_BUCK -> +3V3
- R102 pad 1: /controller/VDD_CTRL -> Net-(U4-BOOT0)
- R102 pad 2: Net-(J6-Pin_3) -> GND
- R133 pad 1: /switch/switch_gpios/JTAG_SWITCH.NTRST -> +3V3
- R84 pad 1: /switch/EN-1V15_STM_TO_BUCK -> +3V3
- R99 pad 1: /switch/EN-2V5_STM_TO_BUCK -> +3V3
- TP11 pad 1: /switch/EN-1V15_STM_TO_BUCK -> +3V3
- TP31 pad 1: /switch/EN-2V5_STM_TO_BUCK -> +3V3
- U2 pad 5: /switch/EN-1V15_STM_TO_BUCK -> +3V3
- U3 pad 5: /switch/EN-2V5_STM_TO_BUCK -> +3V3
- U4 pad 31: /controller/RGMII0_SWITCH_STM.RXCTL-CRS_DV -> /controller/RGMII0_SWITCH_STM.TXCTL-DX_DV
- U4 pad 47: /controller/RGMII0_SWITCH_STM.TXCTL-DX_DV -> Net-(U4-PB11)
- U4 pad 81: /switch/EN-1V15_STM_TO_BUCK -> unconnected-(U4-PD0-Pad81)
- U4 pad 82: /switch/EN-2V5_STM_TO_BUCK -> unconnected-(U4-PD1-Pad82)
- U4 pad 94: Net-(J6-Pin_2) -> Net-(U4-BOOT0)
Routing:
- net /switch/EN-1V15_STM_TO_BUCK: track 117.7 -> 0.00 mm, vias 3 -> 0
- net /switch/EN-2V5_STM_TO_BUCK: track 88.1 -> 0.00 mm, vias 4 -> 0
- net +3V3: track 0.00 -> 68.8 mm
- net Net-(U4-BOOT0): track 0.00 -> 17.3 mm
- net /controller/RGMII0_SWITCH_STM.TXD0: track 41.8 -> 24.9 mm
- net Net-(J6-Pin_2): track 16.2 -> 0.00 mm
- net /controller/RGMII0_SWITCH_STM.TXD1: track 40.0 -> 24.8 mm
- net /controller/RGMII0_SWITCH_STM.TXC-REFCLK: track 38.5 -> 24.3 mm
- net /controller/RGMII0_SWITCH_STM.TXCTL-DX_DV: track 36.8 -> 24.3 mm, vias 2 -> 0
- net /controller/RGMII0_SWITCH_STM.RXCTL-CRS_DV: track 53.8 -> 61.6 mm
- net Net-(J6-Pin_3): track 7.31 -> 0.00 mm
- net Net-(U4-PB11): track 0.00 -> 4.59 mm
- net /controller/RGMII0_SWITCH_STM.RXD1: track 56.8 -> 60.7 mm
- net GND: track 8.26 -> 12.1 mm
- net /controller/RGMII0_SWITCH_STM.RXD0: track 55.5 -> 59.2 mm
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