File: shish-lan.kicad_pcb (KiCad board)
At the start: 6 copper layers, 100 x 100 mm, 305 parts, among them J1 RJ45_0826-1X4T-43-F, J10 Header_07x01_2.54mm_0mm_Strai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, J11 Header_10x02_2.54mm_2.54mm_St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, J13 SMA, J14 SMA, J15 Header_02x01_2.54mm_0mm_Strai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, J16 Header_02x01_2.54mm_0mm_Strai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, J17 Header_02x01_2.54mm_0mm_Strai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, J2 Header_02x01_2.54mm_0mm_Strai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, J3 Header_02x01_2.54mm_0mm_Strai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, J4 Header_03x01_2.54mm_0mm_Strai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, J5 Header_10x02_2.54mm_2.54mm_St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, J7 Header_03x01_2.54mm_0mm_Strai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, J8 Header_02x01_2.54mm_0mm_Strai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, J9 Header_07x01_2.54mm_0mm_Strai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, U1 LAN96455F-I/8MW, U2 TPS564257DRLR, U3 TPS564257DRLR, U4 STM32H742VGT6, U5 TPS564257DRLR, X1 25M, X2 25M

Commit message: PCB rev B: DNP sync, RMII GND vias, R102 silk
Refs #108
Routing:
- net GND: vias 180 -> 185
