File: jtag_header_arm.kicad_sch (KiCad schematic)
At the start: 7 parts, among them J5 Header_10x02_2.54mm_2.54mm_St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

Commit message: Fit R97/R109 for ST-LINK VDD sense
Refs #96
Parts:
- R109, R97: now fitted
Changed lines of the file:
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@@
 		(on_board yes)
 		(in_pos_files yes)
-		(dnp yes)
+		(dnp no)
 		(fields_autoplaced yes)
 		(property "Reference" "R109"
@@
 		(on_board yes)
 		(in_pos_files yes)
-		(dnp yes)
+		(dnp no)
 		(fields_autoplaced yes)
 		(property "Reference" "R97"
